Commit message: add an omni dummy

File: omni_description/xacro/omni.urdf.xacro (robot description, xacro)
@@ -7,5 +7,5 @@
 	<!-- import all gazebo-customization elements, including gazebo colors -->
 	<xacro:include filename="$(find omni_description)/xacro/main.plugin.xacro" />
-	<link name="origin_link"/>
+	<!--link name="origin_link"/-->
 	<link name="base_link">
 	<inertial>
@@ -34,5 +34,5 @@
 	</collision>
 	</link>
-	<joint
+	<!--joint
 		name="base_joint"
 		type="fixed"
@@ -43,5 +43,5 @@
 			xyz="0 0 0.09525"
 		/>
-	</joint>
+	</joint-->
 	<xacro:rim_macro
 		name="left"
