Commit message: use a omni dummy so that no wheel needs to be considered

File: omni_description/xacro/main.plugin.xacro (robot description, xacro)
@@ -30,5 +30,5 @@
 				</noise>
 			</ray>
-			<plugin name="gazebo_ros_head_hokuyo_controller" filename="libgazebo_ros_laser.so">
+			<plugin name="gazebo_ros_head_hokuyo_controller1" filename="libgazebo_ros_laser.so">
 				<topicName>/scan1</topicName>
 				<frameName>/laser_1</frameName>
@@ -64,5 +64,5 @@
 				</noise>
 			</ray>
-			<plugin name="gazebo_ros_head_hokuyo_controller" filename="libgazebo_ros_laser.so">
+			<plugin name="gazebo_ros_head_hokuyo_controller2" filename="libgazebo_ros_laser.so">
 				<topicName>/scan2</topicName>
 				<frameName>/laser_2</frameName>
@@ -76,5 +76,5 @@
       <legacyModeNS>true</legacyModeNS>
     </plugin>
-  </gazebo> -->
+</gazebo> -->
 <!-- Planar move plugin -->
 <gazebo>
@@ -87,3 +87,14 @@
     </plugin>
   </gazebo>
+<!-- Force sensor plugin -->
+<!--gazebo reference="fs_joint">
+	<provideFeedback>true</provideFeedback>
+</gazebo>
+<gazebo>
+	<plugin name="body_joint_ft_sensor" filename="libgazebo_ros_ft_sensor.so">
+		<updateRate>50.0</updateRate>
+		<topicName>/netft_data</topicName>
+		<jointName>fs_joint</jointName>
+	</plugin>
+</gazebo-->
 </robot>

File: omni_description/xacro/omni_dummy.urdf.xacro (robot description, xacro)
@@ -5,12 +5,12 @@
   <link name="move_base">
     <inertial>
-      <mass value="9.82868080625"/>
+      <mass value="200"/>
       <inertia
-	ixx="0.06362454783"
+	ixx="2.2"
 	ixy="0"
 	ixz="0"
-	iyy="0.06362454783"
+	iyy="2.2"
 	iyz="0"
-	izz="0.12331130197"
+	izz="4.0"
       />
     </inertial>
@@ -36,12 +36,12 @@
   <link name="body">
     <inertial>
-      <mass value="9.82868080625"/>
+      <mass value="10"/>
       <inertia
-	ixx="0.06362454783"
+	ixx="0.19"
 	ixy="0"
 	ixz="0"
-	iyy="0.06362454783"
+	iyy="0.19"
 	iyz="0"
-	izz="0.12331130197"
+	izz="0.11"
       />
     </inertial>
@@ -63,6 +63,38 @@
     <parent link="move_base" />
     <child link="body" />
-    <origin xyz="0 0 0.2"/>
+    <origin xyz="0 0 0.25"/>
   </joint>
+  <!--link name="force_sensor">
+    <inertial>
+      <mass value="1"/>
+      <inertia
+	ixx="0.02"
+	ixy="0"
+	ixz="0"
+	iyy="0.02"
+	iyz="0"
+	izz="0.01"
+      />
+    </inertial>
+    <visual>
+      <geometry>
+	<cylinder length="0.02" radius="0.05"/>
+      </geometry>
+      <material name="black">
+	<color rgba="0 0 0 1"/>
+      </material>
+    </visual>
+    <collision>
+      <geometry>
+	<cylinder length="0.02" radius="0.05"/>
+      </geometry>
+    </collision>
+  </link>
+  <joint name="fs_joint" type="revolute">
+    <parent link="body" />
+    <child link="force_sensor" />
+    <origin xyz="0 0 0.23"/>
+    <limit velocity="6.5" effort="1000" lower="0" upper="0" />
+  </joint-->
   <link name="laser_1">
     <inertial>
@@ -121,3 +153,6 @@
     <material>Gazebo/White</material>
   </gazebo>
+  <!--gazebo reference="force_sensor">
+    <material>Gazebo/Grey</material>
+  </gazebo-->
 </robot>

Commit message: updated lidar position & laser scanning specs

File: omni_description/xacro/main.plugin.xacro (robot description, xacro)
@@ -6,17 +6,17 @@
 			<pose>0 0 0 0 0 0</pose>
 			<visualize>true</visualize>
-			<update_rate>50</update_rate>
+			<update_rate>30</update_rate>
 			<ray>
 				<scan>
 					<horizontal>
-						<samples>360</samples>
-						<resolution>1</resolution>
-						<min_angle>-1.570796</min_angle>
-						<max_angle>1.570796</max_angle>
+						<samples>1440</samples>
+						<resolution>0.0043633</resolution>
+						<min_angle>-2.356194</min_angle>
+						<max_angle>2.356194</max_angle>
 					</horizontal>
 				</scan>
 				<range>
 					<min>0.10</min>
-					<max>10.0</max>
+					<max>50.0</max>
 					<resolution>0.01</resolution>
 				</range>
@@ -40,17 +40,17 @@
 			<pose>0 0 0 0 0 0</pose>
 			<visualize>true</visualize>
-			<update_rate>50</update_rate>
+			<update_rate>30</update_rate>
 			<ray>
 				<scan>
 					<horizontal>
-						<samples>360</samples>
-						<resolution>1</resolution>
-						<min_angle>-1.570796</min_angle>
-						<max_angle>1.570796</max_angle>
+						<samples>1440</samples>
+						<resolution>0.0043633</resolution>
+						<min_angle>-2.356194</min_angle>
+						<max_angle>2.356194</max_angle>
 					</horizontal>
 				</scan>
 				<range>
 					<min>0.10</min>
-					<max>10.0</max>
+					<max>50.0</max>
 					<resolution>0.01</resolution>
 				</range>

File: omni_description/xacro/omni_dummy.urdf.xacro (robot description, xacro)
@@ -118,5 +118,5 @@
   <joint name="laser1_joint" type="fixed">
     <axis xyz="0 1 0" />
-    <origin xyz="0.1 0.05 0.23" rpy="0 0 1.0" />
+    <origin xyz="0.1 0.05 0.23" rpy="0 0 1.57079" />
     <parent link="body" />
     <child link="laser_1" />
@@ -143,5 +143,5 @@
   <joint name="laser2_joint" type="fixed">
     <axis xyz="0 1 0" />
-    <origin xyz="0.1 -0.05 0.23" rpy="0 0 -1.0" />
+    <origin xyz="0.1 -0.05 0.23" rpy="0 0 -1.57079" />
     <parent link="body" />
     <child link="laser_2" />

Commit message: remove unnecessary files

File: omni_description/xacro/main.plugin.xacro (robot description, xacro)
@@ -70,4 +70,23 @@
 		</sensor>
 	</gazebo>
+<!-- Planar move plugin -->
+	 <gazebo reference="move_base">
+	  <sensor name="base_bumper" type="contact">
+	    <always_on>1</always_on>
+	    <update_rate>100</update_rate>
+	    <contact>
+	      <!-- When using ROS Indigo and Gazebo 2.2.3, the name specified here
+	           must be <link name>_collision. -->
+	      <collision>base_link_collision</collision>
+	    </contact>
+	    <plugin filename="libgazebo_ros_bumper.so" name="base_bumper">
+	      <always_on>1</always_on>
+	      <update_rate>100</update_rate>
+	      <frameName>move_base</frameName>
+	      <bumperTopicName>base_bumper</bumperTopicName>
+	    </plugin>
+	  </sensor>
+	  <!--material>Gazebo/Orange</material-->
+	</gazebo>
 <!-- ros control plugin
 <gazebo>
@@ -78,13 +97,13 @@
 </gazebo> -->
 <!-- Planar move plugin -->
-<gazebo>
-    <plugin name="object_controller" filename="libgazebo_ros_planar_move.so">
-      <commandTopic>/omnibase/cmd_vel</commandTopic>
-      <odometryTopic>/odom</odometryTopic>
-      <odometryFrame>odom</odometryFrame>
-      <odometryRate>20.0</odometryRate>
-      <robotBaseFrame>base_link</robotBaseFrame>
-    </plugin>
-  </gazebo>
+	<gazebo>
+	    <plugin name="object_controller" filename="libgazebo_ros_planar_move.so">
+	      <commandTopic>/omnibase/cmd_vel</commandTopic>
+	      <odometryTopic>/odom</odometryTopic>
+	      <odometryFrame>odom</odometryFrame>
+	      <odometryRate>20.0</odometryRate>
+	      <robotBaseFrame>base_link</robotBaseFrame>
+	    </plugin>
+	</gazebo>
 <!-- Force sensor plugin -->
 <!--gazebo reference="fs_joint">

File: omni_description/xacro/omni_dummy.urdf.xacro (robot description, xacro)
@@ -23,5 +23,5 @@
       </material>
     </visual>
-    <collision>
+    <collision name="base_link_collision">
       <geometry>
 	<cylinder length="0.1" radius="0.2"/>

Commit message: update lidar configs

File: omni_description/xacro/main.plugin.xacro (robot description, xacro)
@@ -10,6 +10,5 @@
 				<scan>
 					<horizontal>
-						<samples>1440</samples>
-						<resolution>0.0043633</resolution>
+						<samples>1080</samples>
 						<min_angle>-2.356194</min_angle>
 						<max_angle>2.356194</max_angle>
@@ -17,13 +16,10 @@
 				</scan>
 				<range>
-					<min>0.10</min>
-					<max>50.0</max>
-					<resolution>0.01</resolution>
+					<min>0.05</min>
+					<max>60.0</max>
+					<!--resolution>0.01</resolution-->
 				</range>
 				<noise>
 					<type>gaussian</type>
-					<!-- Noise parameters based on published spec for Hokuyo laser achieving
-						"+-30mm" accuracy at range < 10m. A mean of 0.0m and stddev of 0.01m will
-						put 99.7% of samples within 0.03m of the true reading. -->
 					<mean>0.0</mean>
 					<stddev>0.01</stddev>
@@ -35,5 +31,6 @@
 			</plugin>
 		</sensor>
-	</gazebo><!-- lms100 -->
+	</gazebo>
+<!-- lms100 -->
 	<gazebo reference="laser_2">
 		<sensor type="ray" name="head_hokuyo_sensor2">
@@ -44,6 +41,5 @@
 				<scan>
 					<horizontal>
-						<samples>1440</samples>
-						<resolution>0.0043633</resolution>
+						<samples>1080</samples>
 						<min_angle>-2.356194</min_angle>
 						<max_angle>2.356194</max_angle>
@@ -51,13 +47,10 @@
 				</scan>
 				<range>
-					<min>0.10</min>
-					<max>50.0</max>
-					<resolution>0.01</resolution>
+					<min>0.05</min>
+					<max>60.0</max>
+					<!--resolution>0.01</resolution-->
 				</range>
 				<noise>
 					<type>gaussian</type>
-					<!-- Noise parameters based on published spec for Hokuyo laser achieving
-						"+-30mm" accuracy at range < 10m. A mean of 0.0m and stddev of 0.01m will
-						put 99.7% of samples within 0.03m of the true reading. -->
 					<mean>0.0</mean>
 					<stddev>0.01</stddev>

File: omni_description/xacro/omni.urdf.xacro (robot description, xacro)
@@ -112,5 +112,5 @@
       <origin xyz="0 0 0" rpy="0 0 0" />
       <geometry>
-	<box size="0.1 0.1 0.1" />
+	<mesh filename="package://omni_description/mesh/lms100.dae" />
       </geometry>
     </collision>
@@ -137,5 +137,5 @@
       <origin xyz="0 0 0" rpy="0 0 0" />
       <geometry>
-	<box size="0.1 0.1 0.1" />
+	<mesh filename="package://omni_description/mesh/lms100.dae" />
       </geometry>
     </collision>

Commit message: update to make it compaitable to melodic

File: omni_description/xacro/main.plugin.xacro (robot description, xacro)
@@ -27,6 +27,6 @@
 			</ray>
 			<plugin name="gazebo_ros_head_hokuyo_controller1" filename="libgazebo_ros_laser.so">
-				<topicName>/scan1</topicName>
-				<frameName>/laser_1</frameName>
+				<topicName>scan1</topicName>
+				<frameName>laser_1</frameName>
 			</plugin>
 		</sensor>
@@ -58,6 +58,6 @@
 			</ray>
 			<plugin name="gazebo_ros_head_hokuyo_controller2" filename="libgazebo_ros_laser.so">
-				<topicName>/scan2</topicName>
-				<frameName>/laser_2</frameName>
+				<topicName>scan2</topicName>
+				<frameName>laser_2</frameName>
 			</plugin>
 		</sensor>
@@ -67,5 +67,5 @@
 	  <sensor name="base_bumper" type="contact">
 	    <always_on>1</always_on>
-	    <update_rate>100</update_rate>
+	    <update_rate>20</update_rate>
 	    <contact>
 	      <!-- When using ROS Indigo and Gazebo 2.2.3, the name specified here
@@ -75,5 +75,5 @@
 	    <plugin filename="libgazebo_ros_bumper.so" name="base_bumper">
 	      <always_on>1</always_on>
-	      <update_rate>100</update_rate>
+	      <update_rate>20</update_rate>
 	      <frameName>move_base</frameName>
 	      <bumperTopicName>base_bumper</bumperTopicName>
@@ -93,5 +93,5 @@
 	    <plugin name="object_controller" filename="libgazebo_ros_planar_move.so">
 	      <commandTopic>/omnibase/cmd_vel</commandTopic>
-	      <odometryTopic>/odom</odometryTopic>
+	      <odometryTopic>odom</odometryTopic>
 	      <odometryFrame>odom</odometryFrame>
 	      <odometryRate>20.0</odometryRate>

File: omni_description/xacro/omni.urdf (robot description, URDF)
Before this commit: robot omni_base, 5 links, 4 joints
Links:
- link body: mass 9.82868080625 -> 10
- link laser_1: geometry collision mesh filename=package://omni_description/mesh/lms100.dae; visual mesh filename=package://omni_description/mesh/lms100.dae
- link laser_2: geometry collision mesh filename=package://omni_description/mesh/lms100.dae; visual mesh filename=package://omni_description/mesh/lms100.dae
- link move_base: mass 9.82868080625 -> 200
Joints:
- joint body_joint: origin xyz=0 0 0.2 -> xyz=0 0 0.25
